File: Amp_Circuit_Design_v8 (1).brd (EAGLE design)
At the start: 160 x 100 mm, 46 parts, among them IC1 OPA211HT, IC3 OPA211HT, U1 MAX660M, U2 MIC3490-3.3YM5-TR

Commit message: push
Parts:
- moved JTAG 62.5 mm to (34.3, 67.3), turned to 270 degrees
- moved U$1 44.5 mm to (10.2, 68.6), flipped to the bottom, turned to 0 degrees
- flipped J1 to the bottom, turned to 0 degrees
- flipped J2 to the bottom
