File: Amp_Circuit_Design_v8 (1).brd (EAGLE design)
At the start: 40.6 x 64.4 mm, 58 parts, among them IC1 OPA211HT, IC3 OPA211HT, U1 MAX660M, U2 MIC3490-3.3YM5-TR, Y1 CRYSTAL-3.2X2.54-PIN

Commit message: updates
Parts:
- removed D2: LED_GREEN, led:LEDC2012X110N_FLAT-G
- removed INPUT, IN_TH, IN_TH1: (no value), jumper:JP1
- removed R20: 200\, comma.ai:0603-R
- removed S1: MOMENTARY-SWITCH-SPST-SMD-6.0X3.5MM, SparkFun-Switches:TACTILE_SWITCH_SMD_6.0X3.5MM
- added JP1, JP2: PINHD-1X2, Connector:1X02
- added X1, X2, X3: (no value), adafruit:SMA_EDGELAUNCH
- moved JP3 3.94 mm to (1.91, 61.7)
- moved J3 1.02 mm to (7.62, 30.2)
Connections:
- new net GND1: X1.GND@4
- new net GND2: X1.GND@3
- new net GND3: X1.GND@2
- new net GND4: X1.GND@1
- net GND: now also JP1.2, JP2.2, X2.GND@1, X2.GND@2, X2.GND@3, X2.GND@4, X3.GND@1, X3.GND@2, X3.GND@3, X3.GND@4; no longer D2.C, INPUT.1, IN_TH.1, IN_TH1.1, S1.1
- net N$18: now also X1.P; no longer INPUT.2
- net N$21: now also JP1.1; no longer R20.2
- net N$3: now also X3.P; no longer IN_TH.2
- net N$33: no longer S1.2
- net N$38: now also JP2.1, U$1.13; no longer D2.A, R20.1
- net N$7: now also X2.P; no longer IN_TH1.2
Routing:
- net N$18: track 31.9 -> 60.9 mm, vias 0 -> 2
- net N$7: track 2.69 -> 24.3 mm
- net N$3: track 4.52 -> 23.8 mm
- net N$21: track 3.76 -> 21.1 mm
- net N$38: track 3.21 -> 15.6 mm, vias 0 -> 1
- net N$33: track 45.5 -> 40.1 mm
- net N$34: track 2.97 -> 6.41 mm
- net N$32: track 3.04 -> 4.60 mm
Other:
- board size 40.6 x 64.4 mm -> 40.6 x 74.6 mm
- board text added: "+"
- board text added: "ACCEL"
- board text added: "T1"
- board text added: "T2"
- board text added: "UART"

Commit message: Update Amp_Circuit_Design_v8 (1).brd
Routing:
- net N$33: track 40.1 -> 37.5 mm
- net GND: vias 27 -> 30
Changed lines of the file:
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@@
 <contactref element="JP1" pad="2"/>
 <contactref element="JP2" pad="2"/>
-<wire x1="24.13" y1="73.66" x2="31.560009375" y2="71.12" width="0" layer="19" extent="1-1"/>
-<wire x1="24.13" y1="74.93" x2="24.13" y2="73.66" width="0" layer="19" extent="1-1"/>
-<wire x1="19.47" y1="73.66" x2="24.13" y2="73.66" width="0" layer="19" extent="1-1"/>
-<wire x1="19.47" y1="76.2" x2="19.47" y2="73.66" width="0" layer="19" extent="1-1"/>
-<wire x1="19.47" y1="78.74" x2="19.47" y2="76.2" width="0" layer="19" extent="1-1"/>
-<wire x1="20.359" y1="70.612" x2="19.47" y2="73.66" width="0" layer="19" extent="1-16"/>
-<wire x1="19.05" y1="69.85" x2="20.359" y2="70.612" width="0" layer="19" extent="16-16"/>
-<wire x1="16.51" y1="74.93" x2="19.47" y2="73.66" width="0" layer="19" extent="1-1"/>
-<wire x1="15.24" y1="73.66" x2="16.51" y2="74.93" width="0" layer="19" extent="1-1"/>
-<wire x1="13.41" y1="74.38" x2="15.24" y2="73.66" width="0" layer="19" extent="16-16"/>
-<wire x1="12.91" y1="74.38" x2="13.41" y2="74.38" width="0" layer="19" extent="16-16"/>
-<wire x1="13.65" y1="72.39" x2="13.41" y2="74.38" width="0" layer="19" extent="1-16"/>
-<wire x1="11.85" y1="69.85" x2="13.65" y2="72.39" width="0" layer="19" extent="1-1"/>
-<wire x1="11.85" y1="67.31" x2="11.85" y2="69.85" width="0" layer="19" extent="1-1"/>
-<wire x1="8.04" y1="69.85" x2="11.85" y2="69.85" width="0" layer="19" extent="1-1"/>
-<wire x1="8.04" y1="67.31" x2="8.04" y2="69.85" width="0" layer="19" extent="1-1"/>
-<wire x1="8.04" y1="74.93" x2="12.7" y2="76.2" width="0" layer="19" extent="1-16"/>
-<wire x1="3.81" y1="73.787" x2="8.04" y2="74.93" width="0" layer="19" extent="1-1"/>
-<wire x1="22.059" y1="64.389" x2="19.05" y2="69.85" width="0" layer="19" extent="16-16"/>
-<wire x1="19.05" y1="63.5" x2="22.059" y2="64.389" width="0" layer="19" extent="16-16"/>
-<wire x1="20.32" y1="60.96" x2="19.05" y2="63.5" width="0" layer="19" extent="1-1"/>
-<wire x1="15.875" y1="51.626" x2="20.32" y2="60.96" width="0" layer="19" extent="16-16"/>
-<wire x1="13.335" y1="46.609" x2="15.875" y2="51.626" width="0" layer="19" extent="16-16"/>
-<wire x1="12.7" y1="45.72" x2="13.335" y2="46.609" width="0" layer="19" extent="1-1"/>
-<wire x1="10.961" y1="44.069" x2="12.7" y2="45.72" width="0" layer="19" extent="1-1"/>
-<wire x1="8.382" y1="44.87" x2="10.961" y2="44.069" width="0" layer="19" extent="1-1"/>
-<wire x1="7.62" y1="43.18" x2="8.382" y2="44.87" width="0" layer="19" extent="1-1"/>
-<wire x1="6.35" y1="43.18" x2="7.62" y2="43.18" width="0" layer="19" extent="1-1"/>
-<wire x1="5.08" y1="43.18" x2="6.35" y2="43.18" width="0" layer="19" extent="1-1"/>
-<wire x1="3.81" y1="43.18" x2="5.08" y2="43.18" width="0" layer="19" extent="1-1"/>
-<wire x1="2.54" y1="43.18" x2="3.81" y2="43.18" width="0" layer="19" extent="1-1"/>
-<wire x1="6.35" y1="44.87" x2="6.35" y2="43.18" width="0" layer="19" extent="1-1"/>
-<wire x1="2.286" y1="44.87" x2="2.54" y2="43.18" width="0" layer="19" extent="1-1"/>
-<wire x1="4.318" y1="44.87" x2="3.81" y2="43.18" width="0" layer="19" extent="1-1"/>
-<wire x1="3.71475" y1="39.37" x2="3.81" y2="43.18" width="0" layer="19" extent="1-1"/>
-<wire x1="1.651" y1="38.52" x2="3.71475" y2="39.37" width="0" layer="19" extent="1-1"/>
-<wire x1="10.0838" y1="50.165" x2="13.335" y2="46.609" width="0" layer="19" extent="1-1"/>
-<wire x1="8.89" y1="38.52" x2="7.62" y2="43.18" width="0" layer="19" extent="1-1"/>
-<wire x1="5.1562" y1="50.165" x2="10.0838" y2="50.165" width="0" layer="19" extent="1-1"/>
-<wire x1="4.445" y1="51.626" x2="5.1562" y2="50.165" width="0" layer="19" extent="1-16"/>
-<wire x1="2.525" y1="34.546" x2="1.651" y2="38.52" width="0" layer="19" extent="1-1"/>
-<wire x1="7.62" y1="21.082" x2="6.705" y2="25.906" width="0" layer="19" extent="1-1"/>
-<wire x1="7.62" y1="21.082" x2="7.62" y2="21.082" width="0" layer="19" extent="1-16"/>
-<wire x1="12.28" y1="33.02" x2="7.62" y2="33.451" width="0" layer="19" extent="1-1"/>
-<wire x1="13.97" y1="33.02" x2="12.28" y2="33.02" width="0" layer="19" extent="1-1"/>
-<wire x1="15.24" y1="33.02" x2="13.97" y2="33.02" width="0" layer="19" extent="1-1"/>
-<wire x1="15.24" y1="31.75" x2="15.24" y2="33.02" width="0" layer="19" extent="1-1"/>
-<wire x1="13.97" y1="31.75" x2="13.97" y2="33.02" width="0" layer="19" extent="1-1"/>
-<wire x1="12.28" y1="30.48" x2="13.97" y2="31.75" width="0" layer="19" extent="1-1"/>
-<wire x1="19.05" y1="33.02" x2="15.24" y2="33.02" width="0" layer="19" extent="1-1"/>
-<wire x1="20.32" y1="33.02" x2="19.05" y2="33.02" width="0" layer="19" extent="1-1"/>
-<wire x1="22.86" y1="33.02" x2="20.32" y2="33.02" width="0" layer="19" extent="1-1"/>
-<wire x1="24.13" y1="33.02" x2="22.86" y2="33.02" width="0" layer="19" extent="1-1"/>
-<wire x1="25.527" y1="31.33" x2="24.13" y2="33.02" width="0" layer="19" extent="1-1"/>
-<wire x1="12.28" y1="26.67" x2="12.28" y2="30.48" width="0" layer="19" extent="1-1"/>
-<wire x1="12.7" y1="21.082" x2="7.62" y2="21.082" width="0" layer="19" extent="1-1"/>
-<wire x1="12.7" y1="21.082" x2="12.7" y2="21.082" width="0" layer="19" extent="1-16"/>
-<wire x1="17.78" y1="21.082" x2="12.7" y2="21.082" width="0" layer="19" extent="1-1"/>
-<wire x1="17.78" y1="21.082" x2="17.78" y2="21.082" width="0" layer="19" extent="1-16"/>
-<wire x1="22.86" y1="21.082" x2="17.78" y2="21.082" width="0" layer="19" extent="1-1"/>
-<wire x1="22.86" y1="21.082" x2="22.86" y2="21.082" width="0" layer="19" extent="1-16"/>
-<wire x1="25.527" y1="25.312" x2="22.86" y2="21.082" width="0" layer="19" extent="1-1"/>
-<wire x1="31.75" y1="30.48" x2="25.527" y2="31.33" width="0" layer="19" extent="1-1"/>
-<wire x1="31.75" y1="29.21" x2="31.75" y2="30.48" width="0" layer="19" extent="1-1"/>
-<wire x1="32.385" y1="27.168" x2="31.75" y2="29.21" width="0" layer="19" extent="1-1"/>
-<wire x1="1.905" y1="73.279" x2="4.445" y2="51.626" width="0" layer="19" extent="16-16"/>
-<wire x1="34.315" y1="38.735" x2="31.75" y2="30.48" width="0" layer="19" extent="1-1"/>
-<wire x1="1.905" y1="70.231" x2="2.525" y2="25.906" width="0" layer="19" extent="16-16"/>
+<via x="24.13" y="21.59" extent="1-16" drill="0.35"/>
+<via x="25.4" y="21.59" extent="1-16" drill="0.35"/>
+<via x="26.67" y="21.59" extent="1-16" drill="0.35"/>
 </signal>
 <signal name="N$3">
@@
 <wire x1="16.764" y1="77.089" x2="16.764" y2="76.8265" width="0.254" layer="16"/>
 <wire x1="16.256" y1="76.3185" x2="16.764" y2="76.8265" width="0.254" layer="16"/>
-<wire x1="7.86" y1="76.81" x2="9.74" y2="74.93" width="0.254" layer="1"/>
 </signal>
 <signal name="N$21">
