File: Amp_Circuit_Design_v8 (1).sch (EAGLE design)
At the start: 53 parts, among them IC1 OPA211HT, IC3 OPA211HT, J3 10103594, U1 LT8330HS6TR, U2 MIC3490-3.3YM5-TR

Commit message: added converter
Parts:
- removed C7: 4.7 uF, Capacitor:C_CHIP-0805(2012-METRIC)
- removed C8: 4.7pf, capacitor-wima:C5/2.5
- removed C9: 1uf, capacitor-wima:C5/2.5
- removed D1: DIODE, diode:DIODE_DO-219-AC(SOD323F)
- removed L1: 2.7uH, Eagle_WE-TDC (rev19a):WE-TDC_8018_74489430027
- removed R13, R15: 1M, resistor:R-EU_M0805
- removed R14: 806k, resistor:R-EU_M0805
- removed R9: 191k, resistor:R-EU_M0805
- C1: value 4.7pf -> 150 uF; device capacitor-wima:C5/2.5 -> Capacitor:C_CHIP-0805(2012-METRIC)
- C2: value 1uf -> 150 uF; device capacitor-wima:C5/2.5 -> Capacitor:C_CHIP-0805(2012-METRIC)
- U1: value LT8330HS6TR -> MAX660M; device LT8330HS6TR:LT8330HS6TR -> max660:MAX660M
Connections:
- removed net N$16: C7.1, C8.1, IC1.-V, IC3.-V, L1.1, R13.1
- removed net N$25: C9.1, L1.3, U1.SW
- removed net N$32: C2.1, U1.INTVCC
- removed net N$34: C9.2, D1.A, L1.2
- new net -5V: C2.1, IC1.-V, IC3.-V, U1.OUT
- net +5V: now also U1.V+; no longer C1.1, L1.4, R15.1, U1.VIN
- net GND: now also U1.LV; no longer C1.2, C7.2, D1.C, R14.1, R9.2
- net N$31: now also C1.2, U1.C1-; no longer C8.2, R13.2, R9.1, U1.FBX
- net N$8: now also C1.1, U1.C1+; no longer R14.2, R15.2, U1.EN/UVLO
Other:
- moved on the sheet: C1, C2

Commit message: push
Parts:
- added R13, R9: 5.1k, comma.ai:R0603
- C1: value 150 uF -> 10u; device Capacitor:C_CHIP-0805(2012-METRIC) -> comma.ai:C0603
- J3: value 10103594 -> (none); device Connector_USB:10103594 -> USB-C-Breakout:SPARKFUN-CONNECTORS_USB_C16PIN
Connections:
- new net N$16: J3.CC2, R9.2
- new net N$20: J3.CC1, R13.2
- net +5V: now also J3.VBUS; no longer J3.VCC
- net GND: now also J3.SHLD, R13.1, R9.1
Other:
- moved on the sheet: C1

Commit message: added biasing
Parts:
- added C6: 1u, capacitor-wima:C5/2.5
- added JP3: PINHD-1X2, Connector:PINHD-1X2
- added R14, R15: 100K, resistor:R-EU_M0805
Connections:
- new net N$32: C6.2, R14.1, R15.1, U$1.59
- new net N$48: JP3.1, U$1.35
- new net N$49: JP3.2, U$1.34
- net +5V: now also R14.2
- net GND: now also R15.2
- net N$17: now also C6.1; no longer U$1.59
Changed lines of the file:
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@@
 <part name="R13" library="comma.ai" deviceset="R" device="0603" value="5.1k"/>
 <part name="GND17" library="supply1" library_urn="urn:adsk.eagle:library:371" deviceset="GND" device=""/>
+<part name="C6" library="capacitor-wima" library_urn="urn:adsk.eagle:library:116" deviceset="C" device="5/2.5" package3d_urn="urn:adsk.eagle:package:5426/1" value="1u"/>
+<part name="R14" library="resistor" library_urn="urn:adsk.eagle:library:348" deviceset="R-EU_" device="M0805" package3d_urn="urn:adsk.eagle:package:23556/2" value="100K"/>
+<part name="R15" library="resistor" library_urn="urn:adsk.eagle:library:348" deviceset="R-EU_" device="M0805" package3d_urn="urn:adsk.eagle:package:23556/2" value="100K"/>
+<part name="GND18" library="supply1" library_urn="urn:adsk.eagle:library:371" deviceset="GND" device=""/>
+<part name="P+10" library="supply1" library_urn="urn:adsk.eagle:library:371" deviceset="+5V" device=""/>
+<part name="JP3" library="Connector" deviceset="PINHD-1X2" device="" package3d_urn="urn:adsk.eagle:package:22435/2"/>
 </parts>
 <sheets>
@@
 <attribute name="VALUE" x="-170.18" y="-66.04" size="1.778" layer="96" rot="MR0"/>
 </instance>
-<instance part="GND8" gate="1" x="93.98" y="30.48" smashed="yes" rot="MR0">
-<attribute name="VALUE" x="96.52" y="27.94" size="1.778" layer="96" rot="MR0"/>
-</instance>
-<instance part="GND9" gate="1" x="152.4" y="27.94" smashed="yes" rot="MR0">
-<attribute name="VALUE" x="154.94" y="25.4" size="1.778" layer="96" rot="MR0"/>
+<instance part="GND8" gate="1" x="93.98" y="33.02" smashed="yes" rot="MR0">
+<attribute name="VALUE" x="96.52" y="30.48" size="1.778" layer="96" rot="MR0"/>
+</instance>
+<instance part="GND9" gate="1" x="152.4" y="30.48" smashed="yes" rot="MR0">
+<attribute name="VALUE" x="154.94" y="27.94" size="1.778" layer="96" rot="MR0"/>
 </instance>
 <instance part="C5" gate="G$1" x="-185.42" y="-60.96" smashed="yes" rot="MR90">
@@
 <instance part="GND17" gate="1" x="-200.66" y="-83.82" smashed="yes">
 <attribute name="VALUE" x="-203.2" y="-86.36" size="1.778" layer="96"/>
+</instance>
+<instance part="C6" gate="G$1" x="55.88" y="45.72" smashed="yes" rot="MR90">
+<attribute name="NAME" x="56.261" y="47.244" size="1.778" layer="95" rot="MR90"/>
+<attribute name="VALUE" x="51.181" y="47.244" size="1.778" layer="96" rot="MR90"/>
+</instance>
+<instance part="R14" gate="G$1" x="45.72" y="53.34" smashed="yes" rot="MR90">
+<attribute name="NAME" x="47.2186" y="49.53" size="1.778" layer="95" rot="MR90"/>
+<attribute name="VALUE" x="42.418" y="49.53" size="1.778" layer="96" rot="MR90"/>
+</instance>
+<instance part="R15" gate="G$1" x="45.72" y="38.1" smashed="yes" rot="MR270">
+<attribute name="NAME" x="44.2214" y="41.91" size="1.778" layer="95" rot="MR270"/>
+<attribute name="VALUE" x="49.022" y="41.91" size="1.778" layer="96" rot="MR270"/>
+</instance>
+<instance part="GND18" gate="1" x="45.72" y="27.94" smashed="yes" rot="MR0">
+<attribute name="VALUE" x="48.26" y="25.4" size="1.778" layer="96" rot="MR0"/>
+</instance>
+<instance part="P+10" gate="1" x="45.72" y="63.5" smashed="yes" rot="MR0">
+<attribute name="VALUE" x="48.26" y="58.42" size="1.778" layer="96" rot="MR90"/>
+</instance>
+<instance part="JP3" gate="G$1" x="53.34" y="-15.24" smashed="yes">
+<attribute name="NAME" x="46.99" y="-9.525" size="1.778" layer="95"/>
+<attribute name="VALUE" x="46.99" y="-20.32" size="1.778" layer="96"/>
 </instance>
 </instances>
@@
 <wire x1="142.24" y1="-5.08" x2="144.78" y2="-5.08" width="0.1524" layer="91"/>
 </segment>
+<segment>
+<pinref part="R14" gate="G$1" pin="2"/>
+<wire x1="45.72" y1="58.42" x2="45.72" y2="60.96" width="0.1524" layer="91"/>
+<pinref part="P+10" gate="1" pin="+5V"/>
+</segment>
 </net>
 <net name="GND" class="0">
@@
 <segment>
 <wire x1="86.36" y1="38.1" x2="93.98" y2="38.1" width="0.1524" layer="91"/>
-<wire x1="93.98" y1="38.1" x2="93.98" y2="33.02" width="0.1524" layer="91"/>
+<wire x1="93.98" y1="38.1" x2="93.98" y2="35.56" width="0.1524" layer="91"/>
 <pinref part="GND8" gate="1" pin="GND"/>
 <pinref part="IC3" gate="G$1" pin="+IN"/>
 </segment>
 <segment>
-<wire x1="152.4" y1="35.56" x2="152.4" y2="30.48" width="0.1524" layer="91"/>
+<wire x1="152.4" y1="35.56" x2="152.4" y2="33.02" width="0.1524" layer="91"/>
 <pinref part="GND9" gate="1" pin="GND"/>
 <wire x1="152.4" y1="35.56" x2="147.32" y2="35.56" width="0.1524" layer="91"/>
@@
 <junction x="-200.66" y="-78.74"/>
 </segment>
+<segment>
+<pinref part="R15" gate="G$1" pin="2"/>
+<wire x1="45.72" y1="33.02" x2="45.72" y2="30.48" width="0.1524" layer="91"/>
+<pinref part="GND18" gate="1" pin="GND"/>
+</segment>
 </net>
 <net name="N$3" class="0">
@@
 <net name="N$17" class="0">
 <segment>
-<pinref part="U$1" gate="G$1" pin="59"/>
-<wire x1="-5.08" y1="43.18" x2="-5.08" y2="45.72" width="0.1524" layer="91"/>
-<wire x1="-5.08" y1="45.72" x2="60.96" y2="45.72" width="0.1524" layer="91"/>
 <pinref part="R11" gate="G$1" pin="2"/>
 <wire x1="60.96" y1="66.04" x2="66.04" y2="66.04" width="0.1524" layer="91"/>
@@
 <wire x1="63.5" y1="45.72" x2="60.96" y2="45.72" width="0.1524" layer="91"/>
 <wire x1="60.96" y1="45.72" x2="60.96" y2="66.04" width="0.1524" layer="91"/>
+<wire x1="60.96" y1="45.72" x2="58.42" y2="45.72" width="0.1524" layer="91"/>
 <junction x="60.96" y="45.72"/>
+<pinref part="C6" gate="G$1" pin="1"/>
 </segment>
 </net>
@@
 </segment>
 </net>
+<net name="N$32" class="0">
+<segment>
+<pinref part="C6" gate="G$1" pin="2"/>
+<wire x1="50.8" y1="45.72" x2="45.72" y2="45.72" width="0.1524" layer="91"/>
+<wire x1="45.72" y1="45.72" x2="45.72" y2="48.26" width="0.1524" layer="91"/>
+<wire x1="45.72" y1="45.72" x2="45.72" y2="43.18" width="0.1524" layer="91"/>
+<junction x="45.72" y="45.72"/>
+<pinref part="R14" gate="G$1" pin="1"/>
+<pinref part="R15" gate="G$1" pin="1"/>
+<pinref part="U$1" gate="G$1" pin="59"/>
+<wire x1="-5.08" y1="43.18" x2="-5.08" y2="45.72" width="0.1524" layer="91"/>
+<wire x1="45.72" y1="45.72" x2="-5.08" y2="45.72" width="0.1524" layer="91"/>
+</segment>
+</net>
+<net name="N$48" class="0">
+<segment>
+<pinref part="U$1" gate="G$1" pin="35"/>
+<wire x1="43.18" y1="-12.7" x2="50.8" y2="-12.7" width="0.1524" layer="91"/>
+<pinref part="JP3" gate="G$1" pin="1"/>
+</segment>
+</net>
+<net name="N$49" class="0">
+<segment>
+<pinref part="U$1" gate="G$1" pin="34"/>
+<wire x1="43.18" y1="-15.24" x2="50.8" y2="-15.24" width="0.1524" layer="91"/>
+<pinref part="JP3" gate="G$1" pin="2"/>
+</segment>
+</net>

Commit message: PCB push
Parts:
- removed JP1, JP2: PINHD-1X2, Connector:PINHD-1X2
- removed R17: (no value), Resistor:R_CHIP-0805(2012-METRIC)
- removed R19: 0R, Resistor:R_CHIP-0805(2012-METRIC)
- removed U$4: OPA2333HT, Thermocouple:OPA2333HT
- added C14, C17, C18, C7: 10u, comma.ai:C0603
- added C15, C16, C19, C9: 100n, comma.ai:C0603
- added C20, C21: 22p, comma.ai:C0603
- added C8: 1u, comma.ai:C0603
- added S1: MOMENTARY-SWITCH-SPST-SMD-6.0X3.5MM, SparkFun-Switches:MOMENTARY-SWITCH-SPST-SMD-6.0X3.5MM
- added Y1: CRYSTAL-3.2X2.54-PIN, comma.ai:CRYSTAL-3.2X2.54-PIN
- C10: value 100 nF -> 10u; device Capacitor:C_CHIP-0805(2012-METRIC) -> comma.ai:C0603
- C11: value 10 uF/10 V -> 1u; device Capacitor:C_CHIP-0805(2012-METRIC) -> comma.ai:C0603
- C12: value 10 uF/6.3 V -> 100n; device Capacitor:C_CHIP-0805(2012-METRIC) -> comma.ai:C0603
- C13: device Capacitor:C_CHIP-0805(2012-METRIC) -> comma.ai:C0603
- C2: value 150 uF -> 10u; device Capacitor:C_CHIP-0805(2012-METRIC) -> comma.ai:C0603
- C3, C4, C6: device capacitor-wima:C5/2.5 -> comma.ai:C0603
- C5: value 10nF -> 10uF; device eagle-ltspice:CC1206 -> comma.ai:C0603
- R1, R10, R11, R14, R15, R2, R3, R4, R5, R6, R7, R8: device resistor:R-EU_M0805 -> comma.ai:R0603
- R12: device rcl:R-EU_R4527 -> comma.ai:R0603
- R16: value (none) -> 10; device Resistor:R_CHIP-0805(2012-METRIC) -> comma.ai:R0603
- R18: device Resistor:R_CHIP-0805(2012-METRIC) -> comma.ai:R0603
- R20: value 560R -> 200\; device Resistor:R_CHIP-0805(2012-METRIC) -> comma.ai:R0603
Connections:
- removed net N$32 (its old number): C6.2, R14.1, R15.1, U$1.59
- new net N$17: C6.2, R14.2, R15.1, U$1.59
- new net N$46: C21.2, U$1.9, Y1.2
- net +3V3: now also C12.2, C16.2, JTAG.2, R14.1, R18.2; no longer C12.1, JP1.1, R16.1, R17.2, U$1.62, U$1.64
- net +5V: now also C15.2; no longer R14.2, U$4.+V
- net -5V: now also C7.1, C8.1, C9.1
- net GND: now also C12.1, C13.2, C14.1, C15.1, C16.1, C17.1, C18.2, C19.2, C20.1, C21.1, C7.2, C8.2, C9.2, S1.1, U$1.62, U$2.-V; no longer C13.1, R17.1, U$4.-V
- net N$1: now also U$2.O_B; no longer U$4.O_A
- net N$21: now also U$1.12; no longer JP2.2
- net N$22: now also C14.2; no longer C12.2
- net N$33: now also C13.1, R18.1, S1.2; no longer C13.2, R18.2
- net N$35: now also C20.2, U$1.8, Y1.1; no longer JTAG.2, R19.2
- net N$36: now also C18.1, C19.1, R16.1, U$1.64; no longer JP1.2, R18.1, R19.1
- net N$37: now also C17.2, U$1.11; no longer JP2.1, U$1.12
- net N$6: now also U$2.-INB; no longer U$4.-INA
- net N$7: now also U$2.+INB; no longer U$4.+INA
Other:
- moved on the sheet: C10, C11, C12, C13, C3, C4, C5, C6, IN_TH, IN_TH1, JP3

Commit message: updates
Parts:
- removed D2: LED_GREEN, led:CHIP-FLAT-G_0805
- removed INPUT, IN_TH, IN_TH1: (no value), jumper:JP1E
- removed R20: 200\, comma.ai:R0603
- removed S1: MOMENTARY-SWITCH-SPST-SMD-6.0X3.5MM, SparkFun-Switches:MOMENTARY-SWITCH-SPST-SMD-6.0X3.5MM
- added JP1, JP2: PINHD-1X2, Connector:PINHD-1X2
- added X1, X2, X3: (no value), adafruit:SMACONNECTOR_EDGE
Connections:
- net GND: now also JP1.2, JP2.2, X2.GND1, X2.GND2, X2.GND3, X2.GND4, X3.GND1, X3.GND2, X3.GND3, X3.GND4; no longer D2.C, INPUT.1, IN_TH.1, IN_TH1.1, S1.1
- net N$18: now also X1.ANT; no longer INPUT.2
- net N$21: now also JP1.1; no longer R20.2
- net N$3: now also X3.ANT; no longer IN_TH.2
- net N$33: no longer S1.2
- net N$38: now also JP2.1, U$1.13; no longer D2.A, R20.1
- net N$7: now also X2.ANT; no longer IN_TH1.2
